Commit message: changes to dome2

File: dslurdf/output/dome2.urdf (robot description, URDF)
Before this commit: robot dome2, 15 links, 14 joints
Joints:
- joint base_link_to_imu_link: origin xyz=0.03 0 0.053 rpy=1.5707963267948966 0 3.141592653589793 -> xyz=0.0 0 0.05 rpy=0 0 0
- joint base_link_to_laser: origin xyz=0 0 0.1 rpy=0 0 -1.5707963267948966 -> xyz=-0.15 0 0.1 rpy=0 0 -1.5707963267948966
